File: 555 LED Chaser/555 LED Chaser.sch (KiCad schematic (older format))
At the start: 20 parts, among them J1 Barrel_Jack, U1 LM555, U2 4017

Commit message: Modified traces to be 1mm wide for better vinyl printing
Parts:
- C2: value 0.01μ -> 0.01μF; footprint Capacitor_THT:C_Disc_D3.0mm_W1.6mm_P2.50mm -> Capacitor_THT:C_Disc_D4.3mm_W1.9mm_P5.00mm
Changed lines of the file:
@@
 EESchema Schematic File Version 4
 LIBS:555 LED Chaser-cache
-EELAYER 26 0
+EELAYER 29 0
 EELAYER END
 $Descr A4 11693 8268
@@
 P 2650 4050
 F 0 "C2" H 2765 4096 50  0000 L CNN
-F 1 "0.01μ" H 2765 4005 50  0000 L CNN
-F 2 "Capacitor_THT:C_Disc_D3.0mm_W1.6mm_P2.50mm" H 2688 3900 50  0001 C CNN
+F 1 "0.01μF" H 2765 4005 50  0000 L CNN
+F 2 "Capacitor_THT:C_Disc_D4.3mm_W1.9mm_P5.00mm" H 2688 3900 50  0001 C CNN
 F 3 "~" H 2650 4050 50  0001 C CNN
 	1    2650 4050
@@
 $EndComp
 Wire Wire Line
-	7150 4550 7700 4550
-Wire Wire Line
 	7700 4550 7700 4250
 Connection ~ 7700 4250
-Wire Wire Line
-	6850 4550 5900 4550
 Wire Wire Line
 	5900 4550 5900 4300
@@
 Wire Wire Line
 	3250 1650 5900 1650
+Wire Wire Line
+	5900 4550 6850 4550
+Wire Wire Line
+	7150 4550 7700 4550
 $EndSCHEMATC
